File: ESP32-CAM-SHOOTER.kicad_pcb (KiCad board)
At the start: 2 copper layers, 100 x 100 mm, 12 parts, among them J1 Bornier 3 points, J2 ESP32 Header1, J3 ESP32 Header2, J4 Flash mode, J5 I2C PCA9685, J6 I2C ADS1115, J7 I2C ssd1306, J8 I2C Autre

Commit message: add pca footprint
Parts:
- added J10: MAX9814, Connector_PinSocket_2.54mm:PinSocket_1x05_P2.54mm_Vertical, F.Cu at (126.5, 104.1)
- added J11: Laser sensor, Connector_PinSocket_2.54mm:PinSocket_1x03_P2.54mm_Vertical, F.Cu at (108.0, 116.6)
- added J12: ADS1115, Connector_PinHeader_2.54mm:PinHeader_1x10_P2.54mm_Vertical, F.Cu at (104.9, 84.6)
- added J9: PCA9685, Connector_PinHeader_2.54mm:PinHeader_1x06_P2.54mm_Vertical, F.Cu at (39.1, 100.3)
- J4: footprint Connector_PinSocket_2.54mm:PinSocket_1x02_P2.54mm_Vertical -> Connector_PinHeader_2.54mm:PinHeader_1x02_P2.54mm_Vertical
- J5: value I2C PCA9685 -> I2C SX1509 (16 GPIO); footprint Connector_PinSocket_2.54mm:PinSocket_1x04_P2.54mm_Vertical -> Connector_PinHeader_2.54mm:PinHeader_1x04_P2.54mm_Vertical
- J6: value I2C ADS1115 -> I2C DS3231 RTC; footprint Connector_PinSocket_2.54mm:PinSocket_1x04_P2.54mm_Vertical -> Connector_PinHeader_2.54mm:PinHeader_1x04_P2.54mm_Vertical
- J7: value I2C ssd1306 -> I2C ssd1306 Screen; footprint Connector_PinSocket_2.54mm:PinSocket_1x04_P2.54mm_Vertical -> Connector_PinHeader_2.54mm:PinHeader_1x04_P2.54mm_Vertical
- J8: footprint Connector_PinSocket_2.54mm:PinSocket_1x04_P2.54mm_Vertical -> Connector_PinHeader_2.54mm:PinHeader_1x04_P2.54mm_Vertical
- moved J5 35.8 mm to (125.8, 71.5), turned to 270 degrees
- moved J6 20.9 mm to (125.8, 79.5), turned to 270 degrees
- moved J8 18.4 mm to (125.8, 96.5), turned to 270 degrees
- moved J7 9.95 mm to (125.8, 87.9), turned to 270 degrees
Connections:
- J3 pad 5: Net-(J3-Pad5) -> Net-(J12-Pad1)
- J5 pad 2: Net-(J3-Pad6) -> Net-(J12-Pad1)
- J5 pad 3: Net-(J3-Pad7) -> Net-(J3-Pad6)
- J5 pad 4: Net-(J3-Pad5) -> Net-(J3-Pad7)
- J6 pad 2: Net-(J3-Pad6) -> Net-(J12-Pad1)
- J6 pad 3: Net-(J3-Pad7) -> Net-(J3-Pad6)
- J6 pad 4: Net-(J3-Pad5) -> Net-(J3-Pad7)
- J7 pad 2: Net-(J3-Pad6) -> Net-(J12-Pad1)
- J7 pad 3: Net-(J3-Pad7) -> Net-(J3-Pad6)
- J7 pad 4: Net-(J3-Pad5) -> Net-(J3-Pad7)
- J8 pad 2: Net-(J3-Pad6) -> Net-(J12-Pad1)
- J8 pad 3: Net-(J3-Pad7) -> Net-(J3-Pad6)
- J8 pad 4: Net-(J3-Pad5) -> Net-(J3-Pad7)
Routing:
- net Net-(J12-Pad1): track 0.00 -> 210.5 mm, vias 0 -> 2
- net VCC: track 41.7 -> 129.5 mm
- net Net-(J3-Pad6): track 54.8 -> 122.7 mm
- net Net-(J3-Pad5): track 62.2 -> 0.00 mm
- net Net-(J3-Pad7): track 90.4 -> 119.2 mm
- net Net-(J10-Pad2): track 0.00 -> 21.5 mm
- net Net-(J10-Pad4): track 0.00 -> 19.4 mm
- net Net-(J11-Pad3): track 0.00 -> 17.6 mm
Other:
- board text added: "ADS1115 I2C ADC"
- board text added: "Alimnetation +5V"
- board text added: "ESP32-CAM"
- board text added: "Laser Sensor"
- board text added: "MAX9814 Mic"
- board text added: "PCA9685 16 canaux Servo"
